File: PCB/IRMote.kicad_pcb (KiCad board)
At the start: 2 copper layers, 33.2 x 44.8 mm, 11 parts, among them J1 Conn_01x02, Q1 BC547, SW1 SW_SPDT, SW2 SW_Push, SW3 SW_Push, SW4 SW_Push, U1 XIAO-ESP32-C5-SMD, U2 TSOP382xx

Commit message: Updated a lot of stuff
Parts:
- removed U1: XIAO-ESP32-C5-SMD, New_XIAO_Series_Footprints:XIAO-ESP32-C5-SMD
- added U3: XIAO-ESP32-C3-SMD, New_XIAO_Series_Footprints:XIAO-ESP32-C3-SMD, F.Cu at (134.6, 106.6)
Connections:
- net Net-(J1-Pin_2) renamed /CON_P2
- net Net-(SW1-A) renamed /VBET
- J1 pad 1: Net-(J1-Pin_1) -> GND
- R1 pad 1: Net-(U1-D10) -> /D10
- SW2 pad 2: Net-(U1-D2) -> /S1
- SW3 pad 2: Net-(U1-D3) -> /S2
- SW4 pad 2: Net-(U1-D4) -> /S3
- U2 pad 1: Net-(U1-D1) -> /OUT
Routing:
- net Net-(U1-D1): track 40.8 -> 0.00 mm
- net /OUT: track 0.00 -> 38.1 mm
- net /S3: track 0.00 -> 24.4 mm
- net Net-(U1-D4): track 23.6 -> 0.00 mm
- net /S1: track 0.00 -> 17.9 mm
- net /S2: track 0.00 -> 17.5 mm
- net Net-(U1-D2): track 17.1 -> 0.00 mm
- net Net-(U1-D3): track 16.8 -> 0.00 mm
- net GND: track 26.8 -> 42.6 mm, vias 0 -> 64
- net Net-(J1-Pin_1): track 9.36 -> 0.00 mm
- net /D10: track 0.00 -> 7.86 mm
- net Net-(U1-D10): track 7.31 -> 0.00 mm
- net /VBET: track 27.6 -> 34.6 mm, vias 3 -> 2
Other:
- outline, holes or cut-outs redrawn
- board text added: "IRMote"

Commit message: Polished MORE!!
Parts:
- added M3: MountingHole_3.2mm_M3, MountingHole:MountingHole_3.2mm_M3, F.Cu at (150.5, 113.5)
- added M3: MountingHole_3.2mm_M3, MountingHole:MountingHole_3.2mm_M3, F.Cu at (150.0, 77.2)
Other:
- board size 33.2 x 44.8 mm -> 40.8 x 44.9 mm
