File: PCB/IRMote.kicad_sch (KiCad schematic)
At the start: 11 parts, among them J1 Conn_01x02, Q1 BC547, SW1 SW_SPDT, SW2 SW_Push, SW3 SW_Push, SW4 SW_Push, U1 XIAO-ESP32-C5-SMD, U2 TSOP382xx

Commit message: Updated a lot of stuff
Parts:
- removed U1: XIAO-ESP32-C5-SMD, New_XIAO_Series_Footprints:XIAO-ESP32-C5-SMD, symbol Seeed_Studio_XIAO_Series:XIAO-ESP32-C5-SMD
- added U3: XIAO-ESP32-C3-SMD, New_XIAO_Series_Footprints:XIAO-ESP32-C3-SMD, symbol Seeed_Studio_XIAO_Series:XIAO-ESP32-C3-SMD
Connections:
- net +3.3V: now also U3.12 (3V3_OUT)
- net GND: now also J1.1 (Pin_1), U3.13 (GND), U3.18 (GND), U3.22 (GND)
- net S3: now reaches SW4.2
- net S3: now also U3.5 (D4)
- net D10: now reaches R1.1
- net D10: now also U3.11 (D10)
- net OUT: now reaches U2.1 (OUT)
- net OUT: now also U3.2 (D1)
- net VBET: now reaches R2.2, SW1.1 (A)
- net VBET: now also U3.21 (VBAT)
- net S1: now reaches SW2.2
- net S1: now also U3.3 (D2)
- net S2: now reaches SW3.2
- net S2: now also U3.4 (D3)
- net CON_P2: now reaches J1.2 (Pin_2), SW1.2 (B)
- no-connect marks 16 -> 13
Other:
- moved on the sheet: D1, J1, Q1, R1, R2, SW1, SW2, SW3, SW4, U2

Commit message: Polished MORE!!
Other:
- moved on the sheet: SW2, SW3, SW4
Changed lines of the file:
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@@
 	)
 	(rectangle
-		(start 88.9 81.28)
-		(end 113.03 101.6)
+		(start 80.01 81.28)
+		(end 116.84 101.6)
 		(stroke
 			(width 0)
@@
 	(text "Buttons"
 		(exclude_from_sim no)
-		(at 92.456 80.518 0)
+		(at 83.566 80.518 0)
 		(effects
 			(font
@@
 	(wire
 		(pts
-			(xy 97.79 91.44) (xy 99.06 91.44)
+			(xy 88.9 91.44) (xy 90.17 91.44)
 		)
 		(stroke
@@
 	(wire
 		(pts
-			(xy 97.79 95.25) (xy 99.06 95.25)
+			(xy 88.9 95.25) (xy 90.17 95.25)
 		)
 		(stroke
@@
 	(wire
 		(pts
-			(xy 97.79 99.06) (xy 99.06 99.06)
+			(xy 88.9 99.06) (xy 90.17 99.06)
 		)
 		(stroke
@@
 	)
 	(label "S1"
-		(at 109.22 91.44 0)
+		(at 100.33 91.44 0)
 		(effects
 			(font
@@
 	)
 	(label "S2"
-		(at 109.22 95.25 0)
+		(at 100.33 95.25 0)
 		(effects
 			(font
@@
 	)
 	(label "S3"
-		(at 109.22 99.06 0)
+		(at 100.33 99.06 0)
 		(effects
 			(font
@@
 	(symbol
 		(lib_id "Switch:SW_Push")
-		(at 104.14 99.06 0)
+		(at 95.25 99.06 0)
 		(unit 1)
 		(body_style 1)
@@
 		(in_pos_files yes)
 		(dnp no)
-		(fields_autoplaced yes)
 		(property "Reference" "SW4"
-			(at 104.14 91.44 0)
+			(at 114.3 98.044 0)
 			(show_name no)
 			(do_not_autoplace no)
@@
 		)
 		(property "Value" "SW_Push"
-			(at 104.14 93.98 0)
+			(at 107.188 98.044 0)
 			(show_name no)
 			(do_not_autoplace no)
@@
 		)
 		(property "Footprint" "Button_Switch_THT:SW_PUSH_6mm"
-			(at 104.14 93.98 0)
+			(at 95.25 93.98 0)
 			(hide yes)
 			(show_name no)
@@
 		)
 		(property "Datasheet" ""
-			(at 104.14 93.98 0)
+			(at 95.25 93.98 0)
 			(hide yes)
 			(show_name no)
@@
 		)
 		(property "Description" "Push button switch, generic, two pins"
-			(at 104.14 99.06 0)
+			(at 95.25 99.06 0)
 			(hide yes)
 			(show_name no)
@@
 	(symbol
 		(lib_id "power:GND")
-		(at 97.79 91.44 270)
+		(at 88.9 91.44 270)
 		(unit 1)
 		(body_style 1)
@@
 		(fields_autoplaced yes)
 		(property "Reference" "#PWR07"
-			(at 91.44 91.44 0)
+			(at 82.55 91.44 0)
 			(hide yes)
 			(show_name no)
@@
 		)
 		(property "Value" "GND"
-			(at 93.98 91.4399 90)
+			(at 85.09 91.4399 90)
 			(show_name no)
 			(do_not_autoplace no)
@@
 		)
 		(property "Footprint" ""
-			(at 97.79 91.44 0)
+			(at 88.9 91.44 0)
 			(hide yes)
 			(show_name no)
@@
 		)
 		(property "Datasheet" ""
-			(at 97.79 91.44 0)
+			(at 88.9 91.44 0)
 			(hide yes)
 			(show_name no)
@@
 		)
 		(property "Description" "Power symbol creates a global label with name \"GND\" , ground"
-			(at 97.79 91.44 0)
+			(at 88.9 91.44 0)
 			(hide yes)
 			(show_name no)
@@
 		(in_pos_files yes)
 		(dnp no)
-		(fields_autoplaced yes)
 		(property "Reference" "#FLG01"
 			(at 171.45 83.185 0)
@@
 		)
 		(property "Value" "PWR_FLAG"
-			(at 171.45 86.36 0)
+			(at 175.514 85.852 0)
 			(show_name no)
 			(do_not_autoplace no)
@@
 	(symbol
 		(lib_id "Switch:SW_Push")
-		(at 104.14 91.44 0)
+		(at 95.25 91.44 0)
 		(unit 1)
 		(body_style 1)
@@
 		(in_pos_files yes)
 		(dnp no)
-		(fields_autoplaced yes)
 		(property "Reference" "SW2"
-			(at 104.14 83.82 0)
+			(at 113.792 90.678 0)
 			(show_name no)
 			(do_not_autoplace no)
@@
 		)
 		(property "Value" "SW_Push"
-			(at 104.14 86.36 0)
+			(at 107.188 90.424 0)
 			(show_name no)
 			(do_not_autoplace no)
@@
 		)
 		(property "Footprint" "Button_Switch_THT:SW_PUSH_6mm"
-			(at 104.14 86.36 0)
+			(at 95.25 86.36 0)
 			(hide yes)
 			(show_name no)
@@
 		)
 		(property "Datasheet" ""
-			(at 104.14 86.36 0)
+			(at 95.25 86.36 0)
 			(hide yes)
 			(show_name no)
@@
 		)
 		(property "Description" "Push button switch, generic, two pins"
-			(at 104.14 91.44 0)
+			(at 95.25 91.44 0)
 			(hide yes)
 			(show_name no)
@@
 	(symbol
 		(lib_id "power:GND")
-		(at 97.79 99.06 270)
+		(at 88.9 99.06 270)
 		(unit 1)
 		(body_style 1)
@@
 		(fields_autoplaced yes)
 		(property "Reference" "#PWR09"
-			(at 91.44 99.06 0)
+			(at 82.55 99.06 0)
 			(hide yes)
 			(show_name no)
@@
 		)
 		(property "Value" "GND"
-			(at 93.98 99.0599 90)
+			(at 85.09 99.0599 90)
 			(show_name no)
 			(do_not_autoplace no)
@@
 		)
 		(property "Footprint" ""
-			(at 97.79 99.06 0)
+			(at 88.9 99.06 0)
 			(hide yes)
 			(show_name no)
@@
 		)
 		(property "Datasheet" ""
-			(at 97.79 99.06 0)
+			(at 88.9 99.06 0)
 			(hide yes)
 			(show_name no)
@@
 		)
 		(property "Description" "Power symbol creates a global label with name \"GND\" , ground"
-			(at 97.79 99.06 0)
+			(at 88.9 99.06 0)
 			(hide yes)
 			(show_name no)
@@
 		(in_pos_files yes)
 		(dnp no)
-		(fields_autoplaced yes)
 		(property "Reference" "#FLG02"
 			(at 171.45 75.565 0)
@@
 		)
 		(property "Value" "PWR_FLAG"
-			(at 171.45 72.39 0)
+			(at 177.292 73.914 0)
 			(show_name no)
 			(do_not_autoplace no)
@@
 	(symbol
 		(lib_id "Switch:SW_Push")
-		(at 104.14 95.25 0)
+		(at 95.25 95.25 0)
 		(unit 1)
 		(body_style 1)
@@
 		(in_pos_files yes)
 		(dnp no)
-		(fields_autoplaced yes)
 		(property "Reference" "SW3"
-			(at 104.14 87.63 0)
+			(at 114.046 94.234 0)
 			(show_name no)
 			(do_not_autoplace no)
@@
 		)
 		(property "Value" "SW_Push"
-			(at 104.14 90.17 0)
+			(at 107.188 94.234 0)
 			(show_name no)
 			(do_not_autoplace no)
@@
 		)
 		(property "Footprint" "Button_Switch_THT:SW_PUSH_6mm"
-			(at 104.14 90.17 0)
+			(at 95.25 90.17 0)
 			(hide yes)
 			(show_name no)
@@
 		)
 		(property "Datasheet" ""
-			(at 104.14 90.17 0)
+			(at 95.25 90.17 0)
 			(hide yes)
 			(show_name no)
@@
 		)
 		(property "Description" "Push button switch, generic, two pins"
-			(at 104.14 95.25 0)
+			(at 95.25 95.25 0)
 			(hide yes)
 			(show_name no)
@@
 	(symbol
 		(lib_id "power:GND")
-		(at 97.79 95.25 270)
+		(at 88.9 95.25 270)
 		(unit 1)
 		(body_style 1)
@@
 		(fields_autoplaced yes)
 		(property "Reference" "#PWR08"
-			(at 91.44 95.25 0)
+			(at 82.55 95.25 0)
 			(hide yes)
 			(show_name no)
@@
 		)
 		(property "Value" "GND"
-			(at 93.98 95.2499 90)
+			(at 85.09 95.2499 90)
 			(show_name no)
 			(do_not_autoplace no)
@@
 		)
 		(property "Footprint" ""
-			(at 97.79 95.25 0)
+			(at 88.9 95.25 0)
 			(hide yes)
 			(show_name no)
@@
 		)
 		(property "Datasheet" ""
-			(at 97.79 95.25 0)
+			(at 88.9 95.25 0)
 			(hide yes)
 			(show_name no)
@@
 		)
 		(property "Description" "Power symbol creates a global label with name \"GND\" , ground"
-			(at 97.79 95.25 0)
-			(hide yes)
-			(show_name no)
+			(at 88.9 95.25 0)
+			(hide yes)
+			(show_name no)
